File: high_voltage.kicad_sch (KiCad schematic)
At the start: 27 parts, among them J1 EDGE-SMA, J3 BG306-02-A-2-0400-L-G, Q1 LDA111STR, Q2 RGT16BM65DTL, Q3 AO3422, Q4 AO3422, SW3 TL3301AF160QJ, T1 ATB322524, T2 ATB322524

Commit message: finalized schematic + layout
Parts:
- D3, D4, D5: value SM4005PL-TP -> GOODWORK A7
- R2: value ${ALTIUM_VALUE} -> 360k; PART NUMBER RCHIP-300K-2512 -> RCHIP-300K-2510
Connections:
- net VCC renamed +3V3
Changed lines of the file:
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@@
       (effects (font (size 1.27 1.27)) (justify left bottom))
     )
-    (property "Value" "SM4005PL-TP" (at 64.77 115.57 0)
+    (property "Value" "GOODWORK A7" (at 64.77 115.57 0)
       (effects (font (size 1.27 1.27)) (justify left bottom))
     )
@@
         (path "/3227ed55-0ca5-48b6-9dc2-dcbe4715d7c3/fbf650a8-2c0c-4af6-8b5b-5f7ba6e62b3a"
           (reference "D2") (unit 1)
+        )
+      )
+    )
+  )
+  (symbol (lib_id "power:+3V3") (at 19.05 113.03 0) (unit 1)
+    (in_bom yes) (on_board yes) (dnp no) (fields_autoplaced)
+    (property "Reference" "#PWR01" (at 19.05 116.84 0)
+      (effects (font (size 1.27 1.27)) hide)
+    )
+    (property "Value" "+3V3" (at 19.05 109.22 0)
+      (effects (font (size 1.27 1.27)))
+    )
+    (property "Footprint" "" (at 19.05 113.03 0)
+      (effects (font (size 1.27 1.27)) hide)
+    )
+    (property "Datasheet" "" (at 19.05 113.03 0)
+      (effects (font (size 1.27 1.27)) hide)
+    )
+    (pin "1")
+    (instances
+      (project "picoemp_kicad"
+        (path "/3227ed55-0ca5-48b6-9dc2-dcbe4715d7c3/fbf650a8-2c0c-4af6-8b5b-5f7ba6e62b3a"
+          (reference "#PWR01") (unit 1)
         )
       )
@@
     )
   )
-  (symbol (lib_id "chipshouter-pico-hv-altium-import:VCC") (at 119.38 41.91 180) (unit 1)
-    (in_bom yes) (on_board yes) (dnp no)
-    (property "Reference" "#PWR0104" (at 119.38 41.91 0)
-      (effects (font (size 1.27 1.27)) hide)
-    )
-    (property "Value" "VCC" (at 119.38 38.1 0)
-      (effects (font (size 1.27 1.27)))
-    )
-    (property "Footprint" "" (at 119.38 41.91 0)
-      (effects (font (size 1.27 1.27)) hide)
-    )
-    (property "Datasheet" "" (at 119.38 41.91 0)
-      (effects (font (size 1.27 1.27)) hide)
-    )
-    (pin "")
-    (instances
-      (project "picoemp_kicad"
-        (path "/3227ed55-0ca5-48b6-9dc2-dcbe4715d7c3"
-          (reference "#PWR0104") (unit 1)
-        )
-        (path "/3227ed55-0ca5-48b6-9dc2-dcbe4715d7c3/fbf650a8-2c0c-4af6-8b5b-5f7ba6e62b3a"
-          (reference "#PWR02") (unit 1)
-        )
-      )
-    )
-  )
   (symbol (lib_id "chipshouter-pico-hv-altium-import:root_0_DIODE_SCHOTTKY") (at 26.67 125.73 0) (unit 1)
     (in_bom yes) (on_board yes) (dnp no)
@@
       (effects (font (size 1.27 1.27)) (justify left bottom))
     )
-    (property "Value" "SM4005PL-TP" (at 21.59 130.81 0)
+    (property "Value" "GOODWORK A7" (at 21.59 130.81 0)
       (effects (font (size 1.27 1.27)) (justify left bottom))
     )
@@
         (path "/3227ed55-0ca5-48b6-9dc2-dcbe4715d7c3/fbf650a8-2c0c-4af6-8b5b-5f7ba6e62b3a"
           (reference "D3") (unit 1)
+        )
+      )
+    )
+  )
+  (symbol (lib_id "power:+3V3") (at 119.38 41.91 0) (unit 1)
+    (in_bom yes) (on_board yes) (dnp no) (fields_autoplaced)
+    (property "Reference" "#PWR02" (at 119.38 45.72 0)
+      (effects (font (size 1.27 1.27)) hide)
+    )
+    (property "Value" "+3V3" (at 119.38 38.1 0)
+      (effects (font (size 1.27 1.27)))
+    )
+    (property "Footprint" "" (at 119.38 41.91 0)
+      (effects (font (size 1.27 1.27)) hide)
+    )
+    (property "Datasheet" "" (at 119.38 41.91 0)
+      (effects (font (size 1.27 1.27)) hide)
+    )
+    (pin "1")
+    (instances
+      (project "picoemp_kicad"
+        (path "/3227ed55-0ca5-48b6-9dc2-dcbe4715d7c3/fbf650a8-2c0c-4af6-8b5b-5f7ba6e62b3a"
+          (reference "#PWR02") (unit 1)
         )
       )
@@
     )
   )
-  (symbol (lib_id "chipshouter-pico-hv-altium-import:VCC") (at 19.05 113.03 180) (unit 1)
-    (in_bom yes) (on_board yes) (dnp no)
-    (property "Reference" "#PWR0103" (at 19.05 113.03 0)
-      (effects (font (size 1.27 1.27)) hide)
-    )
-    (property "Value" "VCC" (at 19.05 109.22 0)
-      (effects (font (size 1.27 1.27)))
-    )
-    (property "Footprint" "" (at 19.05 113.03 0)
-      (effects (font (size 1.27 1.27)) hide)
-    )
-    (property "Datasheet" "" (at 19.05 113.03 0)
-      (effects (font (size 1.27 1.27)) hide)
-    )
-    (pin "")
-    (instances
-      (project "picoemp_kicad"
-        (path "/3227ed55-0ca5-48b6-9dc2-dcbe4715d7c3"
-          (reference "#PWR0103") (unit 1)
-        )
-        (path "/3227ed55-0ca5-48b6-9dc2-dcbe4715d7c3/fbf650a8-2c0c-4af6-8b5b-5f7ba6e62b3a"
-          (reference "#PWR01") (unit 1)
-        )
-      )
-    )
-  )
   (symbol (lib_id "chipshouter-pico-hv-altium-import:root_0_DIODE_SCHOTTKY") (at 62.23 173.99 0) (unit 1)
     (in_bom yes) (on_board yes) (dnp no)
@@
       (effects (font (size 1.27 1.27)) (justify left bottom))
     )
-    (property "Value" "SM4005PL-TP" (at 60.706 178.816 0)
+    (property "Value" "GOODWORK A7" (at 60.706 178.816 0)
       (effects (font (size 1.27 1.27)) (justify left bottom))
     )
@@
       (effects (font (size 1.27 1.27)) (justify left bottom))
     )
-    (property "Value" "${ALTIUM_VALUE}" (at 205.486 66.04 0)
+    (property "Value" "360k" (at 205.486 66.04 0)
       (effects (font (size 1.27 1.27)) (justify left bottom))
     )
@@
       (effects (font (size 1.27 1.27)) hide)
     )
-    (property "PART NUMBER" "RCHIP-300K-2512" (at 203.454 57.912 0)
-      (effects (font (size 1.27 1.27)) (justify left bottom) hide)
-    )
+    (property "PART NUMBER" "RCHIP-300K-2510" (at 203.454 57.912 0)
+      (effects (font (size 1.27 1.27)) (justify left bottom) hide)
+    )

Commit message: finishing touches
Parts:
- C3: footprint CKG57N_2220 -> Capacitor_SMD:C_2220_5650Metric
Connections:
- no-connect marks 0 -> 1
Other:
- company: (none) -> Colin O'Flynn
- title: (none) -> High voltage
Changed lines of the file:
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@@
 (kicad_sch (version 20230121) (generator eeschema)
   (paper "A4")
+  (title_block
+    (title "High voltage")
+    (date "2023-03-04")
+    (rev "V1")
+    (company "Colin O'Flynn")
+    (comment 1 "KP: Modified footprint and changed of few passive components")
+  )
   (junction (at 115.57 158.75) (diameter 0) (color 0 0 0 0)
   )
@@
   (junction (at 262.89 100.33) (diameter 0) (color 0 0 0 0)
   )
+  (no_connect (at 153.67 57.15))
   (wire (pts (xy 260.35 100.33) (xy 257.81 100.33))
     (stroke (width 0.254) (type default))
@@
   )
   (text_box "SW3 should be 4.6 to 5.2mm high. If too high will hit shield. If too low will be hard to press. Pn here fits well."
-    (at 168.91 26.67 0) (size -33.02 12.7)
+    (at 135.89 26.67 0) (size 33.02 12.7)
     (stroke (width 0) (type default) (color 0 0 0 1))
     (fill (type color) (color 255 255 150 1))
@@
       (effects (font (size 1.27 1.27)) (justify left bottom))
     )
-    (property "Footprint" "CKG57N_2220" (at 181.61 105.41 0)
-      (effects (font (size 1.27 1.27)) hide)
-    )
+    (property "Footprint" "Capacitor_SMD:C_2220_5650Metric" (at 181.61 105.41 0)
+      (effects (font (size 1.27 1.27)) hide)
+    )
