File: mcu.kicad_sch (KiCad schematic)
At the start: 33 parts, among them Q6 FSS2302S, SW1 ARM, SW2 PULSE, SW4 SW_SPST, U1 RP2040, U2 W25Q128JVSIQ, Y1 X322512MSB4SI

Commit message: finalized schematic + layout
Parts:
- added D10: PICO_LED1, LED_SMD:LED_0603_1608Metric, symbol Device:LED
- added J5: Conn_01x03_Socket, Connector_PinHeader_2.54mm:PinHeader_1x03_P2.54mm_Vertical, symbol Connector:Conn_01x03_Socket
- added J6: Conn_01x08_Socket, Connector_PinSocket_2.54mm:PinSocket_1x08_P2.54mm_Vertical, symbol Connector:Conn_01x08_Socket
- added R20: 1k, Resistor_SMD:R_0603_1608Metric, symbol Device:R
- BZ1: value Buzzer -> MLT-7525
- C4: value 100m -> 100n
Connections:
- net +3V3: now also SW2.1, J6.7 (Pin_7); no longer SW2.2
- net ARMED_LED: now also U1.39 (GPIO27/ADC1)
- net BUZZER: now also U1.18 (GPIO15); no longer U1.6 (GPIO4)
- net GND: now also D10.1 (K), J5.2 (Pin_2), J6.8 (Pin_8)
- net PULSE_BUTTON: now also SW2.2; no longer SW2.1
- net GPIO0: now reaches U1.2 (GPIO0)
- net GPIO0: now also J6.1 (Pin_1)
- net SWCLK: now reaches U1.24 (SWCLK)
- net SWCLK: now also J5.1 (Pin_1)
- net SWDIO: now reaches U1.25 (SWDIO)
- net SWDIO: now also J5.3 (Pin_3)
- net GPIO1: now reaches U1.3 (GPIO1)
- net GPIO1: now also J6.2 (Pin_2)
- net PICO_LED: now reaches U1.37 (GPIO25)
- net PICO_LED: now also R20.1
- net GPIO2: now reaches U1.4 (GPIO2)
- net GPIO2: now also J6.3 (Pin_3)
- net GPIO3: now reaches U1.5 (GPIO3)
- net GPIO3: now also J6.4 (Pin_4)
- net GPIO5: now reaches U1.7 (GPIO5)
- net GPIO5: now also J6.6 (Pin_6)
- new net: D10.2 (A), R20.2
- new net GPIO4: J6.5 (Pin_5), U1.6 (GPIO4)
Other:
- note added: "Debug interface"
- moved on the sheet: D12, D8, D9, R15, R16, R27

Commit message: Small tweaks
Other:
- note added: "GPIO header"
- moved on the sheet: J6
Changed lines of the file:
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@@
+    (stroke (width 0) (type default))
+  )
+  (polyline (pts (xy 317.5 185.42) (xy 407.67 185.42))
     (stroke (width 0) (type default))
   )
@@
     (stroke (width 0) (type default))
   )
-  (wire (pts (xy 349.25 39.37) (xy 361.95 39.37))
+  (wire (pts (xy 350.52 215.9) (xy 363.22 215.9))
     (stroke (width 0) (type default))
   )
@@
     (stroke (width 0) (type default))
   )
-  (wire (pts (xy 344.17 54.61) (xy 344.17 57.15))
+  (wire (pts (xy 345.44 231.14) (xy 345.44 233.68))
     (stroke (width 0) (type default))
   )
@@
     (stroke (width 0) (type default))
   )
-  (wire (pts (xy 344.17 52.07) (xy 361.95 52.07))
+  (wire (pts (xy 345.44 228.6) (xy 363.22 228.6))
     (stroke (width 0) (type default))
   )
@@
     (stroke (width 0) (type default))
   )
+  (polyline (pts (xy 407.67 252.73) (xy 317.5 252.73))
+    (stroke (width 0) (type default))
+  )
   (polyline (pts (xy 248.92 285.75) (xy 248.92 185.42))
     (stroke (width 0) (type default))
@@
     (stroke (width 0) (type default))
   )
+  (polyline (pts (xy 407.67 185.42) (xy 407.67 252.73))
+    (stroke (width 0) (type default))
+  )
   (polyline (pts (xy 317.5 185.42) (xy 317.5 11.43))
     (stroke (width 0) (type default))
@@
     (stroke (width 0) (type default))
   )
-  (wire (pts (xy 344.17 54.61) (xy 361.95 54.61))
+  (wire (pts (xy 345.44 231.14) (xy 363.22 231.14))
     (stroke (width 0) (type default))
   )
@@
     (stroke (width 0) (type default))
   )
-  (wire (pts (xy 349.25 49.53) (xy 361.95 49.53))
+  (wire (pts (xy 350.52 226.06) (xy 363.22 226.06))
     (stroke (width 0) (type default))
   )
@@
     (stroke (width 0) (type default))
   )
-  (wire (pts (xy 349.25 36.83) (xy 361.95 36.83))
+  (wire (pts (xy 350.52 213.36) (xy 363.22 213.36))
     (stroke (width 0) (type default))
   )
@@
     (stroke (width 0) (type default))
   )
-  (wire (pts (xy 349.25 41.91) (xy 361.95 41.91))
+  (wire (pts (xy 350.52 218.44) (xy 363.22 218.44))
     (stroke (width 0) (type default))
   )
@@
     (stroke (width 0) (type default))
   )
-  (wire (pts (xy 349.25 46.99) (xy 361.95 46.99))
+  (wire (pts (xy 350.52 223.52) (xy 363.22 223.52))
     (stroke (width 0) (type default))
   )
@@
     (stroke (width 0) (type default))
   )
-  (wire (pts (xy 349.25 44.45) (xy 361.95 44.45))
+  (wire (pts (xy 350.52 220.98) (xy 363.22 220.98))
     (stroke (width 0) (type default))
   )
@@
     (effects (font (size 1.27 1.27)) (justify left bottom))
   )
+  (text "GPIO header" (at 350.52 196.85 0)
+    (effects (font (size 2.5 2.5)) (justify left bottom))
+  )
   (label "XOUT" (at 290.068 52.07 0) (fields_autoplaced)
     (effects (font (size 1.27 1.27)) (justify left bottom))
@@
     (effects (font (size 1.27 1.27)) (justify right bottom))
   )
-  (label "GPIO1" (at 349.25 39.37 0) (fields_autoplaced)
+  (label "GPIO1" (at 350.52 215.9 0) (fields_autoplaced)
     (effects (font (size 1.27 1.27)) (justify left bottom))
   )
@@
     (effects (font (size 1.27 1.27)) (justify right bottom))
   )
-  (label "GPIO4" (at 349.25 46.99 0) (fields_autoplaced)
+  (label "GPIO4" (at 350.52 223.52 0) (fields_autoplaced)
     (effects (font (size 1.27 1.27)) (justify left bottom))
   )
@@
     (effects (font (size 1.27 1.27)) (justify right bottom))
   )
-  (label "GPIO0" (at 349.25 36.83 0) (fields_autoplaced)
+  (label "GPIO0" (at 350.52 213.36 0) (fields_autoplaced)
     (effects (font (size 1.27 1.27)) (justify left bottom))
   )
@@
     (effects (font (size 1.27 1.27)) (justify left bottom))
   )
-  (label "GPIO5" (at 349.25 49.53 0) (fields_autoplaced)
+  (label "GPIO5" (at 350.52 226.06 0) (fields_autoplaced)
     (effects (font (size 1.27 1.27)) (justify left bottom))
   )
@@
     (effects (font (size 1.27 1.27)) (justify left bottom))
   )
-  (label "GPIO3" (at 349.25 44.45 0) (fields_autoplaced)
+  (label "GPIO3" (at 350.52 220.98 0) (fields_autoplaced)
     (effects (font (size 1.27 1.27)) (justify left bottom))
   )
@@
     (effects (font (size 1.27 1.27)) (justify left bottom))
   )
-  (label "GPIO2" (at 349.25 41.91 0) (fields_autoplaced)
+  (label "GPIO2" (at 350.52 218.44 0) (fields_autoplaced)
     (effects (font (size 1.27 1.27)) (justify left bottom))
   )
@@
     )
   )
-  (symbol (lib_id "power:+3V3") (at 344.17 52.07 0) (unit 1)
-    (in_bom yes) (on_board yes) (dnp no) (fields_autoplaced)
-    (property "Reference" "#PWR065" (at 344.17 55.88 0)
-      (effects (font (size 1.27 1.27)) hide)
-    )
-    (property "Value" "+3V3" (at 344.17 48.26 0)
-      (effects (font (size 1.27 1.27)))
-    )
-    (property "Footprint" "" (at 344.17 52.07 0)
-      (effects (font (size 1.27 1.27)) hide)
-    )
-    (property "Datasheet" "" (at 344.17 52.07 0)
+  (symbol (lib_id "power:+3V3") (at 345.44 228.6 0) (unit 1)
+    (in_bom yes) (on_board yes) (dnp no) (fields_autoplaced)
+    (property "Reference" "#PWR065" (at 345.44 232.41 0)
+      (effects (font (size 1.27 1.27)) hide)
+    )
+    (property "Value" "+3V3" (at 345.44 224.79 0)
+      (effects (font (size 1.27 1.27)))
+    )
+    (property "Footprint" "" (at 345.44 228.6 0)
+      (effects (font (size 1.27 1.27)) hide)
+    )
+    (property "Datasheet" "" (at 345.44 228.6 0)
       (effects (font (size 1.27 1.27)) hide)
     )
@@
     )
   )
-  (symbol (lib_name "GND_4") (lib_id "power:GND") (at 344.17 57.15 0) (unit 1)
-    (in_bom yes) (on_board yes) (dnp no) (fields_autoplaced)
-    (property "Reference" "#PWR064" (at 344.17 63.5 0)
-      (effects (font (size 1.27 1.27)) hide)
-    )
-    (property "Value" "GND" (at 344.17 62.23 0)
-      (effects (font (size 1.27 1.27)))
-    )
-    (property "Footprint" "" (at 344.17 57.15 0)
-      (effects (font (size 1.27 1.27)) hide)
-    )
-    (property "Datasheet" "" (at 344.17 57.15 0)
+  (symbol (lib_name "GND_4") (lib_id "power:GND") (at 345.44 233.68 0) (unit 1)
+    (in_bom yes) (on_board yes) (dnp no) (fields_autoplaced)
+    (property "Reference" "#PWR064" (at 345.44 240.03 0)
+      (effects (font (size 1.27 1.27)) hide)
+    )
+    (property "Value" "GND" (at 345.44 238.76 0)
+      (effects (font (size 1.27 1.27)))
+    )
+    (property "Footprint" "" (at 345.44 233.68 0)
+      (effects (font (size 1.27 1.27)) hide)
+    )
+    (property "Datasheet" "" (at 345.44 233.68 0)
       (effects (font (size 1.27 1.27)) hide)
     )
@@
     )
   )
-  (symbol (lib_id "Connector:Conn_01x08_Socket") (at 367.03 44.45 0) (unit 1)
-    (in_bom yes) (on_board yes) (dnp no) (fields_autoplaced)
-    (property "Reference" "J6" (at 368.3 45.085 0)
-      (effects (font (size 1.27 1.27)) (justify left))
-    )
-    (property "Value" "Conn_01x08_Socket" (at 368.3 47.625 0)
-      (effects (font (size 1.27 1.27)) (justify left))
-    )
-    (property "Footprint" "Connector_PinSocket_2.54mm:PinSocket_1x08_P2.54mm_Vertical" (at 367.03 44.45 0)
-      (effects (font (size 1.27 1.27)) hide)
-    )
-    (property "Datasheet" "~" (at 367.03 44.45 0)
-      (effects (font (size 1.27 1.27)) hide)
-    )
+  (symbol (lib_id "Connector:Conn_01x08_Socket") (at 368.3 220.98 0) (unit 1)
+    (in_bom yes) (on_board yes) (dnp no) (fields_autoplaced)
+    (property "Reference" "J6" (at 369.57 221.615 0)
+      (effects (font (size 1.27 1.27)) (justify left))
+    )
+    (property "Value" "Conn_01x08_Socket" (at 369.57 224.155 0)
+      (effects (font (size 1.27 1.27)) (justify left))
+    )
+    (property "Footprint" "Connector_PinSocket_2.54mm:PinSocket_1x08_P2.54mm_Vertical" (at 368.3 220.98 0)
+      (effects (font (size 1.27 1.27)) hide)
+    )
+    (property "Datasheet" "~" (at 368.3 220.98 0)
+      (effects (font (size 1.27 1.27)) hide)
+    )

Commit message: finishing touches
Parts:
- added R26: 100k, Resistor_SMD:R_0603_1608Metric, symbol Device:R
Connections:
- net BUZZER: now also R26.1
- net GND: now also R26.2
Other:
- company: (none) -> Kevin Pettersson
- title: (none) -> MCU
Changed lines of the file:
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@@
 (kicad_sch (version 20230121) (generator eeschema)
   (paper "A3")
+  (title_block
+    (title "MCU")
+    (date "2023-03-04")
+    (rev "V1")
+    (company "Kevin Pettersson")
+  )
   (junction (at 272.796 44.45) (diameter 0) (color 0 0 0 0)
   )
@@
     (stroke (width 0) (type default))
   )
+  (wire (pts (xy 286.766 52.07) (xy 290.068 52.07))
+    (stroke (width 0) (type default))
+  )
+  (wire (pts (xy 62.23 227.33) (xy 62.23 223.52))
+    (stroke (width 0) (type default))
+  )
+  (polyline (pts (xy 407.67 252.73) (xy 317.5 252.73))
+    (stroke (width 0) (type default))
+  )
+  (polyline (pts (xy 248.92 285.75) (xy 248.92 185.42))
+    (stroke (width 0) (type default))
+  )
+  (wire (pts (xy 129.54 55.88) (xy 120.65 55.88))
+    (stroke (width 0) (type default))
+  )
+  (wire (pts (xy 222.25 129.54) (xy 232.41 129.54))
+    (stroke (width 0) (type default))
+  )
+  (wire (pts (xy 44.45 143.51) (xy 44.45 142.24))
+    (stroke (width 0) (type default))
+  )
+  (wire (pts (xy 228.6 144.78) (xy 232.41 144.78))
+    (stroke (width 0) (type default))
+  )
+  (wire (pts (xy 128.27 73.66) (xy 128.27 76.2))
+    (stroke (width 0) (type default))
+  )
+  (wire (pts (xy 272.796 44.45) (xy 286.766 44.45))
+    (stroke (width 0) (type default))
+  )
+  (wire (pts (xy 87.63 171.45) (xy 87.63 170.18))
+    (stroke (width 0) (type default))
+  )
+  (wire (pts (xy 230.886 50.8) (xy 230.886 52.07))
+    (stroke (width 0) (type default))
+  )
+  (wire (pts (xy 267.97 44.45) (xy 272.796 44.45))
+    (stroke (width 0) (type default))
+  )
+  (wire (pts (xy 129.54 48.26) (xy 120.65 48.26))
+    (stroke (width 0) (type default))
+  )
+  (wire (pts (xy 189.23 129.54) (xy 197.104 129.54))
+    (stroke (width 0) (type default))
+  )
+  (wire (pts (xy 271.78 236.22) (xy 281.94 236.22))
+    (stroke (width 0) (type default))
+  )
   (wire (pts (xy 113.03 242.57) (xy 121.92 242.57))
     (stroke (width 0) (type default))
   )
-  (wire (pts (xy 286.766 52.07) (xy 290.068 52.07))
-    (stroke (width 0) (type default))
-  )
-  (wire (pts (xy 62.23 227.33) (xy 62.23 223.52))
-    (stroke (width 0) (type default))
-  )
-  (polyline (pts (xy 407.67 252.73) (xy 317.5 252.73))
-    (stroke (width 0) (type default))
-  )
-  (polyline (pts (xy 248.92 285.75) (xy 248.92 185.42))
-    (stroke (width 0) (type default))
-  )
-  (wire (pts (xy 129.54 55.88) (xy 120.65 55.88))
-    (stroke (width 0) (type default))
-  )
-  (wire (pts (xy 222.25 129.54) (xy 232.41 129.54))
-    (stroke (width 0) (type default))
-  )
-  (wire (pts (xy 44.45 143.51) (xy 44.45 142.24))
-    (stroke (width 0) (type default))
-  )
-  (wire (pts (xy 228.6 144.78) (xy 232.41 144.78))
-    (stroke (width 0) (type default))
-  )
-  (wire (pts (xy 128.27 73.66) (xy 128.27 76.2))
-    (stroke (width 0) (type default))
-  )
-  (wire (pts (xy 272.796 44.45) (xy 286.766 44.45))
-    (stroke (width 0) (type default))
-  )
-  (wire (pts (xy 87.63 171.45) (xy 87.63 170.18))
-    (stroke (width 0) (type default))
-  )
-  (wire (pts (xy 230.886 50.8) (xy 230.886 52.07))
-    (stroke (width 0) (type default))
-  )
-  (wire (pts (xy 267.97 44.45) (xy 272.796 44.45))
-    (stroke (width 0) (type default))
-  )
-  (wire (pts (xy 129.54 48.26) (xy 120.65 48.26))
-    (stroke (width 0) (type default))
-  )
-  (wire (pts (xy 189.23 129.54) (xy 197.104 129.54))
-    (stroke (width 0) (type default))
-  )
-  (wire (pts (xy 271.78 236.22) (xy 281.94 236.22))
-    (stroke (width 0) (type default))
-  )
   (wire (pts (xy 49.784 91.44) (xy 59.69 91.44))
     (stroke (width 0) (type default))
@@
     (stroke (width 0) (type default))
   )
+  (wire (pts (xy 113.03 243.84) (xy 113.03 242.57))
+    (stroke (width 0) (type default))
+  )
   (wire (pts (xy 76.2 171.45) (xy 76.2 170.18))
     (stroke (width 0) (type default))
@@
   )
   (wire (pts (xy 220.98 52.07) (xy 230.886 52.07))
+    (stroke (width 0) (type default))
+  )
+  (wire (pts (xy 113.03 252.73) (xy 113.03 251.46))
     (stroke (width 0) (type default))
   )
@@
     )
   )
+  (symbol (lib_name "GND_1") (lib_id "power:GND") (at 113.03 252.73 0) (unit 1)
+    (in_bom yes) (on_board yes) (dnp no) (fields_autoplaced)
+    (property "Reference" "#PWR075" (at 113.03 259.08 0)
+      (effects (font (size 1.27 1.27)) hide)
+    )
+    (property "Value" "GND" (at 113.03 257.81 0)
+      (effects (font (size 1.27 1.27)))
+    )
+    (property "Footprint" "" (at 113.03 252.73 0)
+      (effects (font (size 1.27 1.27)) hide)
+    )
+    (property "Datasheet" "" (at 113.03 252.73 0)
+      (effects (font (size 1.27 1.27)) hide)
+    )
+    (pin "1")
+    (instances
+      (project "picoemp_kicad"
+        (path "/3227ed55-0ca5-48b6-9dc2-dcbe4715d7c3/7a73d60b-1200-44ba-88e7-a313c65da933"
+          (reference "#PWR075") (unit 1)
+        )
+      )
+    )
+  )
   (symbol (lib_id "Device:R") (at 282.956 52.07 90) (unit 1)
     (in_bom yes) (on_board yes) (dnp no)
@@
         )
       )
+    )
+  )
+  (symbol (lib_id "Device:R") (at 113.03 247.65 0) (unit 1)
+    (in_bom yes) (on_board yes) (dnp no)
+    (property "Reference" "R26" (at 118.11 246.38 0)
+      (effects (font (size 1.27 1.27)))
+    )
+    (property "Value" "100k" (at 118.11 248.92 0)
+      (effects (font (size 1.27 1.27)))
+    )
+    (property "Footprint" "Resistor_SMD:R_0603_1608Metric" (at 111.252 247.65 90)
+      (effects (font (size 1.27 1.27)) hide)
+    )
+    (property "Datasheet" "~" (at 113.03 247.65 0)
+      (effects (font (size 1.27 1.27)) hide)
+    )
+    (pin "1")
+    (pin "2")
+    (instances
+      (project "picoemp_kicad"
+        (path "/3227ed55-0ca5-48b6-9dc2-dcbe4715d7c3/7a73d60b-1200-44ba-88e7-a313c65da933"
+          (reference "R26") (unit 1)
+        )
+      )
+      (project "Temperature probe rp2040"
+        (path "/460313fe-a917-4c7a-9f7f-e32c88e78d52"
+          (reference "R9") (unit 1)
+        )
+      )
